Commit message: LRF urdf

File: robot_description/urdf/laser_macro.xacro (robot description, xacro)
@@ -1,3 +1,4 @@
 <?xml version="1.0"?>
+<!-- UTM-30LX-EW -->
 <robot name="${robot_name}" xmlns:xacro="http://www.ros.org/wiki/xacro">
  <xacro:macro name="laser_macro" params="parent prefix xyz robot_name">
@@ -11,5 +12,5 @@
        <origin xyz="0 0 0" rpy="0 0 0" />
        <geometry>
-         <cylinder radius="0.02" length="0.06" />
+          <box size="0.062 0.062 0.0875" />
        </geometry>
        <material name="red" />
@@ -18,5 +19,5 @@
        <origin xyz="0 0 0" rpy="0 0 0"/>
        <geometry>
-         <cylinder radius="0.02" length="0.06" />
+          <box size="0.062 0.062 0.0875" />
        </geometry>
      </collision>
@@ -33,6 +34,6 @@
              <samples>400</samples>
              <resolution>1</resolution>
-             <min_angle>${radians(-180)}</min_angle>
-             <max_angle>${radians( 180)}</max_angle>
+             <min_angle>${radians(-135)}</min_angle>
+             <max_angle>${radians( 135)}</max_angle>
            </horizontal>
          </scan>
