Commit message: mdのidをyamlからでなくlaunchからevalを使うように変更

File: robot_description/urdf/4omni/laser_macro.xacro (robot description, xacro)
@@ -2,5 +2,5 @@
 <robot name="${robot_name}" xmlns:xacro="http://www.ros.org/wiki/xacro">
  <xacro:macro name="laser_macro" params="parent prefix xyz robot_name">
-   <joint name="${prefix}_joint" type="fixed">
+    <joint name="${prefix}_joint" type="fixed">
      <parent link="${parent}"/>
      <child  link="${prefix}_link"/>
@@ -26,10 +26,10 @@
      <sensor type="ray" name="${prefix}">
        <pose>0 0 0 0 0 0</pose>
-       <visualize>false</visualize>
-       <update_rate>10</update_rate>
+       <visualize>true</visualize>
+       <update_rate>40</update_rate>
        <ray>
          <scan>
            <horizontal>
-             <samples>400</samples>
+             <samples>720</samples>
              <resolution>1</resolution>
              <min_angle>${radians(-90)}</min_angle>

Commit message: odom_linkを使って動作確認

File: robot_description/urdf/4omni/laser_macro.xacro (robot description, xacro)
@@ -8,20 +8,23 @@
    </joint>
    <link name="${prefix}_link">
-     <visual>
-       <origin xyz="0 0 0" rpy="0 0 0" />
-       <geometry>
-         <cylinder radius="0.02" length="0.06" />
-       </geometry>
-       <material name="red" />
-     </visual>
-     <collision>
-       <origin xyz="0 0 0" rpy="0 0 0"/>
-       <geometry>
-         <cylinder radius="0.02" length="0.06" />
-       </geometry>
-     </collision>
+      <visual name="visual">
+        <geometry>
+          <mesh filename="package://robot_description/stl/hokuyo.dae" />
+        </geometry>
+      </visual>
+      <collision name="collision-base">
+        <pose>0 0 -0.0145 0 0 0</pose>
+        <geometry>
+          <box size="0.05 0.05 0.041"/>
+        </geometry>
+      </collision>
+      <collision name="collision-top">
+        <pose>0 0 0.0205 0 0 0</pose>
+        <geometry>
+          <cylinder length="0.029" radius="0.021"/>
+        </geometry>
+      </collision>
    </link>
    <gazebo reference="${prefix}_link">
-     <material>Gazebo/Red</material>
      <sensor type="ray" name="${prefix}">
        <pose>0 0 0 0 0 0</pose>

File: robot_description/urdf/4omni/model.urdf (robot description, URDF)
Before this commit: robot 4omni, 7 links, 6 joints
Joints:
- joint odom_joint: child odom_link -> base_link; origin xyz=0 -0.331 0.044 rpy=0 0 0 -> xyz=0 0.331 -0.044 rpy=0 0 0; parent base_link -> odom_link

Commit message: LRF反転

File: robot_description/urdf/4omni/laser_macro.xacro (robot description, xacro)
@@ -5,5 +5,5 @@
      <parent link="${parent}"/>
      <child  link="${prefix}_link"/>
-     <origin xyz="${xyz}" rpy="0 0 0"/>
+     <origin xyz="${xyz}" rpy="3.14 0 0"/>
    </joint>
    <link name="${prefix}_link">

File: robot_description/urdf/4omni/model.urdf (robot description, URDF)
Before this commit: robot 4omni, 7 links, 6 joints
Joints:
- joint odom_joint: origin xyz=0 0.331 -0.044 rpy=0 0 0 -> xyz=0 -0.176848 -0.044 rpy=0 0 0
