Commit message: urdfにodom_linkを追加

File: robot_description/urdf/4omni/model.urdf (robot description, URDF)
Before this commit: robot 4omni, 6 links, 5 joints
Links:
- added link odom_link; collision cylinder length=0.06 radius=0.02; visual cylinder length=0.06 radius=0.02
Joints:
- added joint odom_joint: type fixed, parent base_link, child odom_link, origin xyz=0 -0.331 0.044 rpy=0 0 0

Commit message: eband_local_plannerがいい感じ？

File: robot_description/urdf/4omni/model.urdf (robot description, URDF)
Before this commit: robot 4omni, 7 links, 6 joints
Links:
- link body_link: mass 2.0 -> $(arg mass)
