Commit message: rqt_reconfiguration for dwa_local_planner

File: robot_description/urdf/4omni/odm_omni_wheel_set.xacro (robot description, xacro)
@@ -126,39 +126,6 @@
       <origin rpy="0 0 0" xyz="0 0 0"/>
     </joint>
-    <link name="${prefix}_base_link" >
-      <inertial>
-        <mass value="0.010"/>
-        <inertia ixx="0.0001" ixy="0" ixz="0" iyy="0.0001" iyz="0" izz="0.0001"/>
-      </inertial>
-    </link>
-    <joint name="${prefix}_sus_joint" type="prismatic">
-      <parent link="${prefix}_base_link"/>
-      <child  link="${prefix}_sus_link"/>
-      <limit lower="-0.02" upper="0.02" effort="100" velocity="1.0" />
-      <axis xyz="0 0 1"/>
-      <origin xyz="0 0 0" rpy="0 0 0"/>
-      <dynamics damping="0.01"/>
-    </joint>
-    <transmission name="${prefix}_sus_trans">
-      <type>transmission_interface/SimpleTransmission</type>
-      <joint name="${prefix}_sus_joint">
-          <hardwareInterface>hardware_interface/EffortJointInterface</hardwareInterface>
-      </joint>
-      <actuator name="${prefix}_sus_motor">
-        <hardwareInterface>hardware_interface/EffortJointInterface</hardwareInterface>
-        <mechanismReduction>1</mechanismReduction>
-      </actuator>
-    </transmission>
-    <gazebo reference="${prefix}_sus_joint">
-      <kp>50000</kp>
-      <kd>500</kd>
-    </gazebo>
-    <link name="${prefix}_sus_link">
-      <inertial>
-        <mass value="0.010"/>
-        <inertia ixx="0.00001" ixy="0.0" ixz="0.0" iyy="0.00001" iyz="0.0" izz="0.00001"/>
-      </inertial>
-    </link>
-    <xacro:motor prefix="${prefix}_motor" parent="${prefix}_sus_link" />
+    <link name="${prefix}_base_link" />
+    <xacro:motor prefix="${prefix}_motor" parent="${prefix}_base_link" />
     <joint name="${prefix}_housind_joint" type="fixed">
       <parent link="${prefix}_motor_shaft_link"/>
@@ -176,5 +143,5 @@
       <inertial>
         <mass value="0.025"/>
-        <inertia ixx="0.00001" ixy="0" ixz="0" iyy="0.00001" iyz="0" izz="0.00001"/>
+        <inertia ixx="0.0001" ixy="0" ixz="0" iyy="0.0001" iyz="0" izz="0.0001"/>
       </inertial>
     </link>
