Commit message: 覚えてない

File: robot_description/urdf/omni4/model.urdf (robot description, URDF)
Before this commit: robot omni4, 7 links, 6 joints
Links:
- link body_link: geometry collision box size=0.08 0.08 0.02; visual box size=0.08 0.08 0.02

File: robot_description/urdf/omni4/odm_omni_wheel_set1.xacro (robot description, xacro)
@@ -39,5 +39,5 @@
       <mu1 value="2.5" />
       <mu2 value="2.5" />
-      <kp value="5000" />
+      <kp value="10000" />
       <kd value="10" />
       <material>Gazebo/Black</material>

Commit message: おどめとり原点補正量変更

File: robot_description/urdf/omni4/model.urdf (robot description, URDF)
Before this commit: robot omni4, 7 links, 6 joints
Joints:
- joint odom_joint: origin xyz=0 -0.176848 -0.044 rpy=0 0 0 -> xyz=0.3095 0.3095 -0.044 rpy=0 0 0

Commit message: sz_to_rz,rz_to_ts3の軌道追従が出来た

File: robot_description/urdf/omni4/model.urdf (robot description, URDF)
Before this commit: robot omni4, 7 links, 6 joints
Links:
- link odom_link: geometry 
Joints:
- joint odom_joint: origin xyz=0.3095 0.3095 -0.044 rpy=0 0 0 -> xyz=0.0 0.0 -0.0 rpy=0 0 0

File: robot_description/urdf/omni4/odm_omni_wheel_set.xacro (robot description, xacro)
@@ -41,4 +41,6 @@
       <kp value="5000" />
       <kd value="10" />
+      <!-- <kp value="10000" />
+      <kd value="100" /> -->
       <material>Gazebo/Black</material>
     </gazebo>
