Commit message: PoseFollowerを修正してTrajectoryTrackingを作成

File: robot_description/urdf/omni4/laser_macro.xacro (robot description, xacro)
@@ -5,5 +5,5 @@
      <parent link="${parent}"/>
      <child  link="${prefix}_link"/>
-     <origin xyz="${xyz}" rpy="3.14 0 0"/>
+     <origin xyz="${xyz}" rpy="-3.14 0 -1.57"/>
    </joint>
    <link name="${prefix}_link">

Commit message: 青コート用にlaunchに分岐を追加

File: robot_description/urdf/omni4/laser_macro.xacro (robot description, xacro)
@@ -5,5 +5,5 @@
      <parent link="${parent}"/>
      <child  link="${prefix}_link"/>
-     <origin xyz="${xyz}" rpy="-3.14 0 -1.57"/>
+     <origin xyz="${xyz}" rpy="-3.14 0 0"/>
    </joint>
    <link name="${prefix}_link">
@@ -34,5 +34,5 @@
          <scan>
            <horizontal>
-             <samples>720</samples>
+             <samples>180</samples>
              <resolution>1</resolution>
              <min_angle>${radians(-90)}</min_angle>

File: robot_description/urdf/omni4/model.urdf (robot description, URDF)
Before this commit: robot omni4, 7 links, 6 joints
Links:
- added link catch_link, mass 0; collision box size=0.1 0.1 0.02; visual box size=0.1 0.1 0.02
Joints:
- added joint catch_joint: type fixed, parent base_link, child catch_link, origin xyz=0.1 -0.1 0.2 rpy=0 1.57 2.35619
